File: maglev2025_hardware_test2/untitled.kicad_sch (KiCad schematic)
At the start: 21 parts, among them J3 Conn_01x04, J4 Conn_01x04_MountingPin, J5 USB_C_Receptacle_USB2.0

Commit message: finish test2 sche
Parts:
- added C82, C83, C84: 100n, Capacitor_SMD:C_0603_1608Metric, symbol Device:C
- added D29, D30, D31: LED, LED_SMD:LED_0603_1608Metric, symbol Device:LED
- added J6: Conn_01x04, Connector_PinHeader_2.54mm:PinHeader_1x04_P2.54mm_Vertical, symbol Connector_Generic:Conn_01x04
- added R37, R38, R39, R40: 33r, Resistor_SMD:R_0603_1608Metric, symbol Device:R
- added R41, R44, R47: 330, Resistor_SMD:R_0603_1608Metric, symbol Device:R
- added R42, R45, R48: 1k, Resistor_SMD:R_0603_1608Metric, symbol Device:R
- added R43, R46, R49: 10k, Resistor_SMD:R_0603_1608Metric, symbol Device:R
- added SW1, SW2, SW3: ~, 0_RM2023:Button_Hoz, symbol 0_RM2023:SW_Push_MP
- J3: footprint (none) -> Connector_PinHeader_2.54mm:PinHeader_1x04_P2.54mm_Vertical
Connections:
- net +3.3V: now also R42.1, R43.1, R45.1, R46.1, R48.1, R49.1
- net GND: now also C82.1, C83.1, C84.1, SW1.2, SW1.3 (MP), SW2.2, SW2.3 (MP), SW3.2, SW3.3 (MP)
- new net: D31.1 (K), R47.1, R49.2, SW3.1
- new net: D29.2 (A), R42.2
- new net: D29.1 (K), R41.1, R43.2, SW1.1
- new net: J6.1 (Pin_1), R37.2
- new net: J6.2 (Pin_2), R38.2
- new net: J6.3 (Pin_3), R39.2
- new net: J6.4 (Pin_4), R40.2
- new net: D30.1 (K), R44.1, R46.2, SW2.1
- new net: D31.2 (A), R48.2
- new net: D30.2 (A), R45.2
- new net PC10: R38.1
- new net PC11: R39.1
- new net PC12: R40.1
- new net PC13: C82.2, C83.2, C84.2, R41.2, R44.2, R47.2
- new net PD2: R37.1
Other:
- note added: "EXTEND GPIO"

Commit message: Fix on test 2 schematic
Parts:
- removed C54, C56, C82, C83, C84: 100n, Capacitor_SMD:C_0603_1608Metric, symbol Device:C
- removed D29, D30, D31: LED, LED_SMD:LED_0603_1608Metric, symbol Device:LED
- removed D4: DSS34, Diode_SMD:D_SMA, symbol Device:D_Schottky
- removed R43, R46, R49: 10k, Resistor_SMD:R_0603_1608Metric, symbol Device:R
- removed R44, R47: 330, Resistor_SMD:R_0603_1608Metric, symbol Device:R
- removed R45, R48: 1k, Resistor_SMD:R_0603_1608Metric, symbol Device:R
- removed SW1, SW2, SW3: ~, 0_RM2023:Button_Hoz, symbol 0_RM2023:SW_Push_MP
- added C85, C86, C87, C88: 100n, Capacitor_SMD:C_0603_1608Metric, symbol Device:C
- added D4: DK5V45R10, Diode_SMD:D_PowerDI-5, symbol Device:D
- added R50, R52, R55: 10k, Resistor_SMD:R_0603_1608Metric, symbol Device:R
- added R51, R53, R54: 33, Resistor_SMD:R_0603_1608Metric, symbol Device:R
- added SW4: RotaryEncoder_Switch_MP, Rotary_Encoder:RotaryEncoder_Alps_EC11E-Switch_Vertical_H20mm_MountingHoles, symbol Device:RotaryEncoder_Switch_MP
- R41: value 330 -> 5.1k
- R42: value 1k -> 5.1k
Connections:
- net PC13 is gone; now on net UCPD1_CC1: R41.2
- net +3.3V: now also R50.1, R52.1, R55.1; no longer C55.1, J4.3 (Pin_3), R42.1
- net GND: now also R41.1, R42.1, C85.1, C86.1, C87.1, C88.1, SW4.C, SW4.MP, SW4.S2
- net UCPD1_CC2: now also R42.2
- net VPP: now also D4.1 (K)
- net VSENSE_VBUS: now also C88.2
- net at F3.2: now also D4.2 (A)
- new net: R50.2, R51.2, SW4.S1
- new net: R52.2, R53.2, SW4.A
- new net: R54.2, R55.2, SW4.B
- new net +5V: C55.1, J4.3 (Pin_3)
- new net PB10_ROTENC_BTN: C85.2, R51.1
- new net PC6_T8C1: C86.2, R53.1
- new net PC7_T8C2: C87.2, R54.1
Other:
- note added: "I2C OLED Display"
- note removed: "I2C TFT Display"

Commit message: addjust layout
Parts:
- removed C55, C85, C86, C87, C88: 100n, Capacitor_SMD:C_0603_1608Metric, symbol Device:C
- removed C57: 10n, Capacitor_SMD:C_0603_1608Metric, symbol Device:C
- removed D4: DK5V45R10, Diode_SMD:D_PowerDI-5, symbol Device:D
- removed F3: 5A, Fuse:Fuse_1206_3216Metric, symbol Device:Fuse
- removed J3, J6: Conn_01x04, Connector_PinHeader_2.54mm:PinHeader_1x04_P2.54mm_Vertical, symbol Connector_Generic:Conn_01x04
- removed J4: Conn_01x04_MountingPin, Connector_JST:JST_GH_BM04B-GHS-TBT_1x04-1MP_P1.25mm_Vertical, symbol Connector_Generic_MountingPin:Conn_01x04_MountingPin
- removed J5: USB_C_Receptacle_USB2.0, Connector_USB:USB_C_Receptacle_HRO_TYPE-C-31-M-12, symbol Connector:USB_C_Receptacle_USB2.0
- removed R21, R22, R25, R26, R28, R29, R37, R38, R39, R40: 33r, Resistor_SMD:R_0603_1608Metric, symbol Device:R
- removed R23, R24: 4.7k, Resistor_SMD:R_0603_1608Metric, symbol Device:R
- removed R27: 1M, Resistor_SMD:R_0603_1608Metric, symbol Device:R
- removed R30: R_US, Resistor_SMD:R_2512_6332Metric, symbol Device:R_US
- removed R31, R50, R52, R55: 10k, Resistor_SMD:R_0603_1608Metric, symbol Device:R
- removed R32: 1k, Resistor_SMD:R_0603_1608Metric, symbol Device:R
- removed R41, R42: 5.1k, Resistor_SMD:R_0603_1608Metric, symbol Device:R
- removed R51, R53, R54: 33, Resistor_SMD:R_0603_1608Metric, symbol Device:R
- removed SW4: RotaryEncoder_Switch_MP, Rotary_Encoder:RotaryEncoder_Alps_EC11E-Switch_Vertical_H20mm_MountingHoles, symbol Device:RotaryEncoder_Switch_MP
Connections:
- no-connect marks 6 -> 0
Other:
- note removed: "EXTEND GPIO"
- note removed: "I2C OLED Display"
- note removed: "UART"
- note removed: "UCPD"
