File: maglev2025_hardware_sensor/maglev2025_hardware_sensor.kicad_pcb (KiCad board)
At the start: 2 copper layers, 16 x 16 mm, 8 parts, among them J8 Conn_01x07_MountingPin, U2 TMAG5170-Q1

Commit message: solve merge problem
Parts:
- removed J8: Conn_01x07_MountingPin, Connector_JST:JST_GH_SM07B-GHS-TB_1x07-1MP_P1.25mm_Horizontal
- added J9: Conn_01x07_MountingPin, Connector_JST:JST_GH_SM07B-GHS-TB_1x07-1MP_P1.25mm_Horizontal, B.Cu at (8.10, 7.95)
Routing:
- net +3.3V: track 3.77 -> 9.31 mm, vias 3 -> 5
- net SPI1_SCK: track 4.39 -> 2.73 mm
- net SPI1_MISO: track 4.33 -> 2.91 mm
- net ~{MAG_CS}: track 3.17 -> 4.30 mm
- net GND: vias 77 -> 70
Other:
- board text added: "TMAG5170"
- board text added: "X"
- board text added: "Y"
- board text added: "Z"
